File: cores/proto-core/hardware/kicad/ProtoCore_v1.kicad_pcb (KiCad board)
At the start: 6 copper layers, 25 x 25 mm, 91 parts, among them U1 ESP32-S3R8, U10 BMP390, U2 TPS62902RPJR, U3 TPS22810DRV, U4 TPS3899DL30DSER, U5 M24C02-FMH6TG, U6 W25Q128JVP, U7 EMMC04G-CT32_4-Line, U8 LSM6DSO32TR, Y1 CM8V-T1A-32.768KHZ-7PF-20PPM-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

Commit message: minor updates
Parts:
- R7: value 22R -> 499R
Changed lines of the file:
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@@
 			)
 		)
-		(property "Value" "22R"
+		(property "Value" "499R"
 			(at -0.025 2.25 90)
 			(layer "F.Fab")
